File: noleds.sch (KiCad schematic (older format))
At the start: 34 parts, among them P1 USB, P2 CONN_01X03, SW0:0 SWITCH_DIODE, SW0:1 SWITCH_DIODE, SW0:2 SWITCH_DIODE, SW0:3 SWITCH_DIODE, SW0:4 SWITCH_DIODE, SW0:5 SWITCH_DIODE, SW0:6 SWITCH_DIODE, SW1:0 SWITCH_DIODE, SW1:1 SWITCH_DIODE, SW1:2 SWITCH_DIODE, SW1:3 SWITCH_DIODE, SW1:4 SWITCH_DIODE, SW1:5 SWITCH_DIODE, SW2:0 SWITCH_DIODE, SW2:1 SWITCH_DIODE, SW2:2 SWITCH_DIODE, SW2:3 SWITCH_DIODE, SW2:4 SWITCH_DIODE, SW2:5 SWITCH_DIODE, SW2:6 SWITCH_DIODE, SW3:0 SWITCH_DIODE, SW3:1 SWITCH_DIODE, SW3:2 SWITCH_DIODE, SW3:3 SWITCH_DIODE, SW3:4 SWITCH_DIODE, SW3:5 SWITCH_DIODE, SW3:6 SWITCH_DIODE, SW4:5 SWITCH_DIODE, SW4:6 SWITCH_DIODE

Commit message: Add proper 3.5mm jack pins
Parts:
- removed SWR1: SW_PUSH, Buttons_Switches_ThroughHole:SW_Tactile_SPST_Angled, symbol SW_PUSH
- P2: footprint Keyboards:3mmJack -> Pin_Headers:Pin_Header_Angled_1x03
Connections:
- net ROW1: no longer SW2:6.4 (K)
- net ROW2: now also SW2:6.4 (K)
Other:
- moved on the sheet: SW2:6
Changed lines of the file:
@@
 F 0 "P2" H 3650 1400 50  0000 C CNN
 F 1 "CONN_01X03" V 3750 1200 50  0000 C CNN
-F 2 "Keyboards:3mmJack" H 3650 1200 50  0001 C CNN
+F 2 "Pin_Headers:Pin_Header_Angled_1x03" H 3650 1200 50  0001 C CNN
 F 3 "" H 3650 1200 50  0000 C CNN
 	1    3650 1200
@@
 L SWITCH_DIODE SW2:6
 U 1 1 56ED6EBF
-P 6000 4850
-F 0 "SW2:6" H 6000 4650 60  0000 C CNN
-F 1 "SWITCH_DIODE" H 6000 4750 39  0000 C CNN
-F 2 "Keyboards:MX_FLIP_DIODE" H 6000 4850 60  0001 C CNN
-F 3 "" H 6000 4850 60  0000 C CNN
-	1    6000 4850
+P 6000 5450
+F 0 "SW2:6" H 6000 5250 60  0000 C CNN
+F 1 "SWITCH_DIODE" H 6000 5350 39  0000 C CNN
+F 2 "Keyboards:MX_FLIP_DIODE" H 6000 5450 60  0001 C CNN
+F 3 "" H 6000 5450 60  0000 C CNN
+	1    6000 5450
 	1    0    0    -1
 $EndComp
@@
 Wire Wire Line
 	1800 5900 6600 5900
+Wire Wire Line
+	6300 5500 6300 5450
+Connection ~ 5700 5450
+Connection ~ 6300 5900
 $Comp
 L SWITCH_DIODE SW3:0
@@
 $EndComp
 $Comp
-L GND #PWR07
+L GND #PWR08
 U 1 1 56F1AFF1
 P 3200 1100
-F 0 "#PWR07" H 3200 850 50  0001 C CNN
+F 0 "#PWR08" H 3200 850 50  0001 C CNN
 F 1 "GND" H 3200 950 50  0000 C CNN
 F 2 "" H 3200 1100 50  0000 C CNN
@@
 	1    0    0    -1
 $EndComp
-$Comp
-L SW_PUSH SWR1
-U 1 1 572E2571
-P 4550 2500
-F 0 "SWR1" H 4700 2610 50  0000 C CNN
-F 1 "SW_PUSH" H 4550 2420 50  0000 C CNN
-F 2 "Buttons_Switches_ThroughHole:SW_Tactile_SPST_Angled" H 4550 2500 50  0001 C CNN
-F 3 "" H 4550 2500 50  0000 C CNN
-	1    4550 2500
-	1    0    0    -1
-$EndComp
-$Comp
-L Earth #PWR08
-U 1 1 572E3FEC
-P 4850 2500
-F 0 "#PWR08" H 4850 2250 50  0001 C CNN
-F 1 "Earth" H 4850 2350 50  0001 C CNN
-F 2 "" H 4850 2500 50  0000 C CNN
-F 3 "" H 4850 2500 50  0000 C CNN
-	1    4850 2500
-	0    -1   -1   0
-$EndComp
-Text Label 4000 2500 0    60   ~ 0
-RST
-Wire Wire Line
-	4000 2500 4250 2500
-Wire Wire Line
-	6300 4850 6300 4900
-Connection ~ 6300 5300
-Connection ~ 5700 4850
 $EndSCHEMATC
