File: schbackup.sch (KiCad schematic (older format))
At the start: 34 parts, among them P1 USB, P2 CONN_01X03, SW0:0 SWITCH_DIODE, SW0:1 SWITCH_DIODE, SW0:2 SWITCH_DIODE, SW0:3 SWITCH_DIODE, SW0:4 SWITCH_DIODE, SW0:5 SWITCH_DIODE, SW0:6 SWITCH_DIODE, SW1:0 SWITCH_DIODE, SW1:1 SWITCH_DIODE, SW1:2 SWITCH_DIODE, SW1:3 SWITCH_DIODE, SW1:4 SWITCH_DIODE, SW1:5 SWITCH_DIODE, SW2:0 SWITCH_DIODE, SW2:1 SWITCH_DIODE, SW2:2 SWITCH_DIODE, SW2:3 SWITCH_DIODE, SW2:4 SWITCH_DIODE, SW2:5 SWITCH_DIODE, SW2:6 SWITCH_DIODE, SW3:0 SWITCH_DIODE, SW3:1 SWITCH_DIODE, SW3:2 SWITCH_DIODE, SW3:3 SWITCH_DIODE, SW3:4 SWITCH_DIODE, SW3:5 SWITCH_DIODE, SW3:6 SWITCH_DIODE, SW4:5 SWITCH_DIODE, SW4:6 SWITCH_DIODE

Commit message: Add proper 3.5mm jack pins
Parts:
- removed P1: USB, Keyboards:USBMINI, symbol USB_OTG
- removed SWR1: SW_PUSH, Buttons_Switches_ThroughHole:SW_Tactile_SPST_Angled, symbol SW_PUSH
- removed UW1: USBWireConnection, Keyboards:USBWirePins, symbol USBWireConnection
- added D30, D31, D32, D33, D34, D35, D36: LED, LEDs:LED_1206, symbol LED
- added P1: USB_A, Keyboards:MUSB-X151-XX, symbol USB_A
- added R1, R2, R3, R4, R5, R6, R7: 100R, Resistors_SMD:R_2512_HandSoldering, symbol R
- P2: footprint Keyboards:3mmJack -> Pin_Headers:Pin_Header_Angled_1x03
- SW4:5, SW4:6: footprint Keyboards:MX_FLIP_DIODE -> (none)
Connections:
- net labels added: LED+
- net labels removed: Earth, RST
- wire segments 53 -> 49
- no-connect marks 1 -> 6
Other:
- moved on the sheet: SW2:6
