File: Microdox.kicad_pcb (KiCad board)
At the start: 2 copper layers, 153.3 x 135.5 mm, 38 parts, among them P1 USB, P2 CONN_01X03

Commit message: Update?
Honestly I have no idea what I changed ._.
Parts:
- moved ? 1.42 mm to (71.8, 83.2)
Connections:
- ? pad 1: (no net) -> GND (x4)
Routing:
- net /COL2: track 142.0 -> 149.4 mm
- net /SER: track 80.1 -> 82.9 mm
- net Net-(SW0:2-Pad2): track 10.7 -> 13.2 mm
- net Net-(P1-Pad1): track 126.4 -> 127.2 mm
- net /ROW1: track 231.0 -> 231.7 mm
- net Net-(SW3:2-Pad2): track 13.8 -> 13.1 mm
- net Net-(SW3:1-Pad2): track 13.8 -> 13.1 mm
- net Net-(SW3:3-Pad2): track 13.8 -> 13.1 mm
- net Net-(SW2:3-Pad2): track 13.8 -> 13.1 mm
- net Net-(SW1:3-Pad2): track 13.8 -> 13.1 mm
- net /COL6: track 169.5 -> 170.1 mm
Other:
- board text added: "Microdox PCB // v1.0"
- board text added: "The Microdox PCB // v1.0"
